Commit message: Make antbot_real self-contained with STEP model

File: src/antbot_description/urdf/antbot.xacro (robot description, xacro)
@@ -1,6 +1,6 @@
 <?xml version="1.0" ?>
 <!--
-  UMR-style visual conversion built on the validated ANTBot 4WS/4WD skeleton.
-  The package and all eight actuated joint names remain unchanged.
+  GK4XC-001-003 CAD visual on the validated ANTBot 4WS/4WD skeleton.
+  The package, sensor/control TF frames and all eight actuated joint names remain unchanged.
 -->
 <robot name="antbot" xmlns:xacro="http://ros.org/wiki/xacro">
@@ -24,30 +24,23 @@
   <xacro:include filename="$(find antbot_description)/urdf/base.xacro"/>
   <xacro:include filename="$(find antbot_description)/urdf/wheel.xacro"/>
-  <xacro:include filename="$(find antbot_description)/urdf/payload_tower.xacro"/>
   <xacro:include filename="$(find antbot_description)/urdf/ros2_control.xacro"/>
-  <!-- Photo/datasheet-based first-pass geometry -->
-  <xacro:property name="overall_length" value="0.830"/>
-  <xacro:property name="overall_width" value="0.540"/>
-  <xacro:property name="overall_height" value="0.410"/>
-  <xacro:property name="body_height" value="0.410"/>
-  <!-- Wheel proportions inferred from the supplied orthogonal/oblique views -->
-  <xacro:property name="wheelbase_length" value="0.530"/>
-  <xacro:property name="wheel_center_track" value="0.480"/>
-  <xacro:property name="steering_width" value="0.360"/>
-  <xacro:property name="wheel_radius" value="0.080"/>
+  <!-- Measured from the supplied SolidWorks STEP assembly. -->
+  <xacro:property name="overall_length" value="0.5510"/>
+  <xacro:property name="overall_width" value="0.8186"/>
+  <xacro:property name="overall_height" value="1.2861"/>
+  <xacro:property name="body_height" value="1.2861"/>
+  <!-- Measured wheel centres: the four module axes are the vertices of a
+       330 mm square, centred on base_link. -->
+  <xacro:property name="wheelbase_length" value="0.330"/>
+  <xacro:property name="wheel_center_track" value="0.330"/>
+  <xacro:property name="steering_width" value="0.330"/>
+  <xacro:property name="wheel_radius" value="0.0525"/>
   <xacro:property name="wheel_width" value="0.058"/>
   <xacro:property name="steering_height" value="${wheel_radius}"/>
   <xacro:property name="wheel_offset" value="${(wheel_center_track - steering_width)/2}"/>
-  <!-- Existing wheel mesh is 205.943 mm diameter and 75.2 mm wide -->
-  <xacro:property name="wheel_mesh_scale" value="0.000777"/>
-  <xacro:property name="steering_mesh_scale" value="0.000750"/>
-  <!--
-    The top collision reaches z=0.410 m.  With the lidar mount at z=0.344 m,
-    0.070 m puts the optical scan plane at z=0.414 m: clear of the top collision
-    while remaining visually attached to the 0.038 m-high dome.
-  -->
+  <!-- Preserve the existing calibrated scan-frame offset. The chassis STEP
+       does not define ROS sensor frames, so those transforms are unchanged. -->
   <xacro:property name="lidar_scan_z_offset" value="0.070"/>
   <xacro:Base/>
-  <xacro:PayloadTower/>
   <xacro:SwerveWheelLeft position_name="front_left"
                          x_pos="${wheelbase_length/2}" y_pos="${steering_width/2}"/>
@@ -58,5 +51,5 @@
   <xacro:SwerveWheelRight position_name="rear_right"
                           x_pos="${-wheelbase_length/2}" y_pos="${-steering_width/2}"/>
-  <!-- Approximate UMR sensor frames; refine after hardware measurements -->
+  <!-- Sensor TF frames are retained independently from the CAD visual. -->
   <xacro:Sensors name="camera_stereo_front_depth" xyz="0.410 0.045 0.205" rpy="0.0 0.0 0.0"/>
   <xacro:OpticalFrame name="camera_stereo_front_depth_optical" parent="camera_stereo_front_depth"/>

File: src/antbot_description/urdf/base.xacro (robot description, xacro)
@@ -1,7 +1,10 @@
 <?xml version="1.0" ?>
 <!--
-  UMR concept-v2 body.  Visual details are intentionally richer than the
-  collision model; all control joints and frames remain compatible.
-  base_link origin: ground plane, +X front, +Y left, +Z up.
+  GK4XC-001-003 production chassis visual.
+  The source STEP is authored in millimetres. The generated STL is centred
+  around its source axes. In the supplied assembly CAD +X is the installed
+  vertical direction, so a -90 degree ROS Y rotation puts the wheel platform
+  on the floor with its column and manipulator above the chassis.
+  Keep collision geometry simple: the detailed mesh is visual-only.
 -->
 <robot name="base" xmlns:xacro="http://ros.org/wiki/xacro">
@@ -13,140 +16,21 @@
         <inertia ixx="2.56" ixy="0" ixz="0" iyy="5.14" iyz="0" izz="6.37"/>
       </inertial>
-      <!-- Rounded/tapered black lower chassis: z=0.095..0.275 m -->
       <visual>
-        <origin xyz="0 0 0.185" rpy="0 0 0"/>
-        <geometry><mesh filename="package://antbot_description/meshes/umr_lower_body.stl"/></geometry>
-        <material name="umr_dark"/>
+        <origin xyz="0.2754 0 0.6430" rpy="0 -1.57079632679 0"/>
+        <geometry>
+          <mesh filename="package://antbot_description/meshes/gk4xc_001_003_full.stl"
+                scale="0.001 0.001 0.001"/>
+        </geometry>
+        <material name="gk4xc_metal">
+          <color rgba="0.66 0.69 0.73 1.0"/>
+        </material>
       </visual>
-      <!-- White shoulder shell: broad at the bottom and tapered toward the roof -->
-      <visual>
-        <origin xyz="0 0 0.300" rpy="0 0 0"/>
-        <geometry><mesh filename="package://antbot_description/meshes/umr_upper_shell.stl"/></geometry>
-        <material name="umr_white"><color rgba="0.94 0.95 0.96 1.0"/></material>
-      </visual>
-      <!-- Black raised equipment box and white top payload plate -->
-      <visual>
-        <origin xyz="0 0 0.357" rpy="0 0 0"/>
-        <geometry><mesh filename="package://antbot_description/meshes/umr_black_riser.stl"/></geometry>
-        <material name="umr_black"/>
-      </visual>
-      <visual>
-        <origin xyz="0 0 0.390" rpy="0 0 0"/>
-        <geometry><mesh filename="package://antbot_description/meshes/umr_top_plate.stl"/></geometry>
-        <material name="umr_white"><color rgba="0.94 0.95 0.96 1.0"/></material>
-      </visual>
-      <!-- Large white trapezoid service doors on both sides -->
-      <visual>
-        <origin xyz="0 0.266 0" rpy="0 0 0"/>
-        <geometry><mesh filename="package://antbot_description/meshes/umr_side_service_panel.stl"/></geometry>
-        <material name="umr_white"><color rgba="0.94 0.95 0.96 1.0"/></material>
-      </visual>
-      <visual>
-        <origin xyz="0 -0.266 0" rpy="0 0 0"/>
-        <geometry><mesh filename="package://antbot_description/meshes/umr_side_service_panel.stl"/></geometry>
-        <material name="umr_white"><color rgba="0.94 0.95 0.96 1.0"/></material>
-      </visual>
-      <!-- Front/rear white fascia and black center recesses -->
-      <visual>
-        <origin xyz="0.414 0 0" rpy="0 0 0"/>
-        <geometry><mesh filename="package://antbot_description/meshes/umr_front_fascia.stl"/></geometry>
-        <material name="umr_white"><color rgba="0.94 0.95 0.96 1.0"/></material>
-      </visual>
-      <visual>
-        <origin xyz="-0.414 0 0" rpy="0 0 ${pi}"/>
-        <geometry><mesh filename="package://antbot_description/meshes/umr_front_fascia.stl"/></geometry>
-        <material name="umr_white"><color rgba="0.94 0.95 0.96 1.0"/></material>
-      </visual>
-      <visual>
-        <origin xyz="0.412 0 0" rpy="0 0 0"/>
-        <geometry><mesh filename="package://antbot_description/meshes/umr_front_recess.stl"/></geometry>
-        <material name="umr_black"/>
-      </visual>
-      <visual>
-        <origin xyz="-0.412 0 0" rpy="0 0 ${pi}"/>
-        <geometry><mesh filename="package://antbot_description/meshes/umr_front_recess.stl"/></geometry>
-        <material name="umr_black"/>
-      </visual>
-      <!-- Blue corner light bars with black bezels, front and rear -->
-      <xacro:property name="face_x" value="0.420"/>
-      <xacro:property name="light_y" value="0.176"/>
-      <visual><origin xyz="${face_x} ${light_y} 0.296"/><geometry><box size="0.014 0.128 0.028"/></geometry><material name="umr_black"/></visual>
-      <visual><origin xyz="${face_x} ${light_y} 0.296"/><geometry><box size="0.016 0.108 0.012"/></geometry><material name="umr_blue"/></visual>
-      <visual><origin xyz="${face_x} ${-light_y} 0.296"/><geometry><box size="0.014 0.128 0.028"/></geometry><material name="umr_black"/></visual>
-      <visual><origin xyz="${face_x} ${-light_y} 0.296"/><geometry><box size="0.016 0.108 0.012"/></geometry><material name="umr_blue"/></visual>
-      <visual><origin xyz="${-face_x} ${light_y} 0.296"/><geometry><box size="0.014 0.128 0.028"/></geometry><material name="umr_black"/></visual>
-      <visual><origin xyz="${-face_x} ${light_y} 0.296"/><geometry><box size="0.016 0.108 0.012"/></geometry><material name="umr_blue"/></visual>
-      <visual><origin xyz="${-face_x} ${-light_y} 0.296"/><geometry><box size="0.014 0.128 0.028"/></geometry><material name="umr_black"/></visual>
-      <visual><origin xyz="${-face_x} ${-light_y} 0.296"/><geometry><box size="0.016 0.108 0.012"/></geometry><material name="umr_blue"/></visual>
-      <!-- Thin side accent lights, visible in top view -->
-      <visual><origin xyz="0 0.272 0.296"/><geometry><box size="0.105 0.014 0.027"/></geometry><material name="umr_black"/></visual>
-      <visual><origin xyz="0 0.274 0.296"/><geometry><box size="0.086 0.015 0.011"/></geometry><material name="umr_blue"/></visual>
-      <visual><origin xyz="0 -0.272 0.296"/><geometry><box size="0.105 0.014 0.027"/></geometry><material name="umr_black"/></visual>
-      <visual><origin xyz="0 -0.274 0.296"/><geometry><box size="0.086 0.015 0.011"/></geometry><material name="umr_blue"/></visual>
-      <!-- Front/rear vertical dual-lens corner sensor pods -->
-      <xacro:property name="pod_y" value="0.205"/>
-      <xacro:property name="pod_z1" value="0.180"/>
-      <xacro:property name="pod_z2" value="0.220"/>
-      <xacro:macro name="front_pod" params="x y direction">
-        <visual><origin xyz="${x} ${y} 0.200"/><geometry><box size="0.016 0.055 0.095"/></geometry><material name="umr_black"/></visual>
-        <visual><origin xyz="${x + direction*0.010} ${y} ${pod_z1}" rpy="0 ${pi/2} 0"/><geometry><cylinder radius="0.012" length="0.006"/></geometry><material name="metal_silver"/></visual>
-        <visual><origin xyz="${x + direction*0.014} ${y} ${pod_z1}" rpy="0 ${pi/2} 0"/><geometry><cylinder radius="0.007" length="0.004"/></geometry><material name="sensor_glass"/></visual>
-        <visual><origin xyz="${x + direction*0.010} ${y} ${pod_z2}" rpy="0 ${pi/2} 0"/><geometry><cylinder radius="0.012" length="0.006"/></geometry><material name="metal_silver"/></visual>
-        <visual><origin xyz="${x + direction*0.014} ${y} ${pod_z2}" rpy="0 ${pi/2} 0"/><geometry><cylinder radius="0.007" length="0.004"/></geometry><material name="sensor_glass"/></visual>
-      </xacro:macro>
-      <xacro:front_pod x="0.416" y="${pod_y}" direction="1"/>
-      <xacro:front_pod x="0.416" y="${-pod_y}" direction="1"/>
-      <xacro:front_pod x="-0.416" y="${pod_y}" direction="-1"/>
-      <xacro:front_pod x="-0.416" y="${-pod_y}" direction="-1"/>
-      <!-- Paired horizontal center camera modules on front and rear -->
-      <xacro:macro name="center_camera_pair" params="x direction">
-        <visual><origin xyz="${x} 0.055 0.200"/><geometry><box size="0.017 0.072 0.034"/></geometry><material name="umr_deep_black"/></visual>
-        <visual><origin xyz="${x} -0.055 0.200"/><geometry><box size="0.017 0.072 0.034"/></geometry><material name="umr_deep_black"/></visual>
-        <visual><origin xyz="${x + direction*0.011} 0.036 0.200"/><geometry><sphere radius="0.0045"/></geometry><material name="sensor_glass"/></visual>
-        <visual><origin xyz="${x + direction*0.011} 0.055 0.200"/><geometry><sphere radius="0.0045"/></geometry><material name="sensor_glass"/></visual>
-        <visual><origin xyz="${x + direction*0.011} 0.074 0.200"/><geometry><sphere radius="0.0045"/></geometry><material name="sensor_glass"/></visual>
-        <visual><origin xyz="${x + direction*0.011} -0.036 0.200"/><geometry><sphere radius="0.0045"/></geometry><material name="sensor_glass"/></visual>
-        <visual><origin xyz="${x + direction*0.011} -0.055 0.200"/><geometry><sphere radius="0.0045"/></geometry><material name="sensor_glass"/></visual>
-        <visual><origin xyz="${x + direction*0.011} -0.074 0.200"/><geometry><sphere radius="0.0045"/></geometry><material name="sensor_glass"/></visual>
-      </xacro:macro>
-      <xacro:center_camera_pair x="0.420" direction="1"/>
-      <xacro:center_camera_pair x="-0.420" direction="-1"/>
-      <!-- Slanted ventilation slots on both side panels -->
-      <xacro:macro name="vent_group" params="y side_sign x_center angle">
-        <visual><origin xyz="${x_center-0.035} ${y} 0.247" rpy="0 ${angle} 0"/><geometry><box size="0.048 0.014 0.011"/></geometry><material name="umr_black"/></visual>
-        <visual><origin xyz="${x_center} ${y} 0.247" rpy="0 ${angle} 0"/><geometry><box size="0.048 0.014 0.011"/></geometry><material name="umr_black"/></visual>
-        <visual><origin xyz="${x_center+0.035} ${y} 0.247" rpy="0 ${angle} 0"/><geometry><box size="0.048 0.014 0.011"/></geometry><material name="umr_black"/></visual>
-      </xacro:macro>
-      <xacro:vent_group y="0.273" side_sign="1" x_center="0.270" angle="${radians(35)}"/>
-      <xacro:vent_group y="0.273" side_sign="1" x_center="-0.270" angle="${radians(-35)}"/>
-      <xacro:vent_group y="-0.273" side_sign="-1" x_center="0.270" angle="${radians(35)}"/>
-      <xacro:vent_group y="-0.273" side_sign="-1" x_center="-0.270" angle="${radians(-35)}"/>
-      <!-- Subtle panel seams and fasteners on the front/rear fascia -->
-      <visual><origin xyz="0.421 0.168 0.301"/><geometry><box size="0.010 0.003 0.056"/></geometry><material name="panel_seam"/></visual>
-      <visual><origin xyz="0.421 -0.168 0.301"/><geometry><box size="0.010 0.003 0.056"/></geometry><material name="panel_seam"/></visual>
-      <visual><origin xyz="-0.421 0.168 0.301"/><geometry><box size="0.010 0.003 0.056"/></geometry><material name="panel_seam"/></visual>
-      <visual><origin xyz="-0.421 -0.168 0.301"/><geometry><box size="0.010 0.003 0.056"/></geometry><material name="panel_seam"/></visual>
-      <xacro:macro name="fascia_screw" params="x y direction">
-        <visual><origin xyz="${x + direction*0.008} ${y} 0.276" rpy="0 ${pi/2} 0"/><geometry><cylinder radius="0.0045" length="0.004"/></geometry><material name="metal_silver"/></visual>
-      </xacro:macro>
-      <xacro:fascia_screw x="0.420" y="0.125" direction="1"/>
-      <xacro:fascia_screw x="0.420" y="0" direction="1"/>
-      <xacro:fascia_screw x="0.420" y="-0.125" direction="1"/>
-      <xacro:fascia_screw x="-0.420" y="0.125" direction="-1"/>
-      <xacro:fascia_screw x="-0.420" y="0" direction="-1"/>
-      <xacro:fascia_screw x="-0.420" y="-0.125" direction="-1"/>
-      <!-- Simplified collision hulls: no decorative details -->
-      <collision><origin xyz="0 0 0.185"/><geometry><box size="0.780 0.480 0.180"/></geometry></collision>
-      <collision><origin xyz="0 0 0.305"/><geometry><box size="0.700 0.420 0.145"/></geometry></collision>
-      <collision><origin xyz="0 0 0.390"/><geometry><box size="0.660 0.450 0.040"/></geometry></collision>
+      <!-- Conservative envelope for planning; never use the CAD mesh itself
+           as a real-time collision shape. -->
+      <collision>
+        <origin xyz="0 0 0.6430" rpy="0 0 0"/>
+        <geometry><box size="0.5510 0.8186 1.2861"/></geometry>
+      </collision>
     </link>
-    <material name="umr_white"><color rgba="0.94 0.95 0.96 1.0"/></material>
-    <material name="umr_dark"><color rgba="0.085 0.090 0.100 1.0"/></material>
-    <material name="umr_black"><color rgba="0.025 0.030 0.036 1.0"/></material>
-    <material name="umr_deep_black"><color rgba="0.010 0.013 0.018 1.0"/></material>
-    <material name="umr_blue"><color rgba="0.075 0.40 1.00 1.0"/></material>
-    <material name="metal_silver"><color rgba="0.66 0.69 0.73 1.0"/></material>
-    <material name="sensor_glass"><color rgba="0.025 0.070 0.120 1.0"/></material>
-    <material name="panel_seam"><color rgba="0.38 0.40 0.43 1.0"/></material>
   </xacro:macro>
 </robot>

File: src/antbot_description/urdf/wheel.xacro (robot description, xacro)
@@ -1,26 +1,11 @@
 <?xml version="1.0" ?>
-<!-- Four independent steering + drive modules, with concept-style silver hubs. -->
+<!--
+  Four independent steering + drive kinematic modules.
+  Their visible hardware is already part of the all-in-one GK4XC STEP mesh, so
+  these links intentionally contain collision and inertia only.
+-->
 <robot name="wheel" xmlns:xacro="http://ros.org/wiki/xacro">
-  <xacro:macro name="WheelHub" params="face_y">
-    <visual><origin xyz="0 ${face_y} 0" rpy="${pi/2} 0 0"/><geometry><cylinder radius="0.056" length="0.009"/></geometry><material name="hub_silver"/></visual>
-    <visual><origin xyz="0 ${face_y*1.05} 0" rpy="${pi/2} 0 0"/><geometry><cylinder radius="0.038" length="0.010"/></geometry><material name="hub_light"/></visual>
-    <visual><origin xyz="0 ${face_y*1.10} 0" rpy="${pi/2} 0 0"/><geometry><cylinder radius="0.017" length="0.012"/></geometry><material name="hub_silver"/></visual>
-    <!-- eight fixed hub bolts; explicit coordinates avoid nested-macro scope issues -->
-    <visual><origin xyz="0.047 ${face_y*1.12} 0" rpy="${pi/2} 0 0"/><geometry><cylinder radius="0.0032" length="0.006"/></geometry><material name="hub_bolt_dark"/></visual>
-    <visual><origin xyz="0.033234 ${face_y*1.12} 0.033234" rpy="${pi/2} 0 0"/><geometry><cylinder radius="0.0032" length="0.006"/></geometry><material name="hub_bolt_dark"/></visual>
-    <visual><origin xyz="0 ${face_y*1.12} 0.047" rpy="${pi/2} 0 0"/><geometry><cylinder radius="0.0032" length="0.006"/></geometry><material name="hub_bolt_dark"/></visual>
-    <visual><origin xyz="-0.033234 ${face_y*1.12} 0.033234" rpy="${pi/2} 0 0"/><geometry><cylinder radius="0.0032" length="0.006"/></geometry><material name="hub_bolt_dark"/></visual>
-    <visual><origin xyz="-0.047 ${face_y*1.12} 0" rpy="${pi/2} 0 0"/><geometry><cylinder radius="0.0032" length="0.006"/></geometry><material name="hub_bolt_dark"/></visual>
-    <visual><origin xyz="-0.033234 ${face_y*1.12} -0.033234" rpy="${pi/2} 0 0"/><geometry><cylinder radius="0.0032" length="0.006"/></geometry><material name="hub_bolt_dark"/></visual>
-    <visual><origin xyz="0 ${face_y*1.12} -0.047" rpy="${pi/2} 0 0"/><geometry><cylinder radius="0.0032" length="0.006"/></geometry><material name="hub_bolt_dark"/></visual>
-    <visual><origin xyz="0.033234 ${face_y*1.12} -0.033234" rpy="${pi/2} 0 0"/><geometry><cylinder radius="0.0032" length="0.006"/></geometry><material name="hub_bolt_dark"/></visual>
-  </xacro:macro>
   <xacro:macro name="SwerveWheelLeft" params="position_name x_pos y_pos">
     <link name="${position_name}_steering_link">
-      <visual>
-        <origin xyz="0 0 0" rpy="0 0 ${pi}"/>
-        <geometry><mesh filename="package://antbot_description/meshes/steering_link_r.stl" scale="${steering_mesh_scale} ${steering_mesh_scale} ${steering_mesh_scale}"/></geometry>
-        <material name="metal_gray"/>
-      </visual>
       <collision><origin xyz="0 -0.020 0.035"/><geometry><box size="0.050 0.075 0.110"/></geometry></collision>
       <inertial><mass value="1.0"/><origin xyz="0 -0.020 0.035"/><inertia ixx="0.0017" ixy="0" ixz="0" iyy="0.0014" iyz="0" izz="0.0008"/></inertial>
@@ -32,6 +17,4 @@
     </joint>
     <link name="${position_name}_wheel_link">
-      <visual><origin rpy="0 0 ${pi}"/><geometry><mesh filename="package://antbot_description/meshes/wheel_link_r.stl" scale="${wheel_mesh_scale} ${wheel_mesh_scale} ${wheel_mesh_scale}"/></geometry><material name="tire_black"/></visual>
-      <xacro:WheelHub face_y="0.035"/>
       <collision><origin rpy="${pi/2} 0 0"/><geometry><cylinder radius="${wheel_radius}" length="${wheel_width}"/></geometry></collision>
       <inertial><mass value="2.0"/><inertia ixx="0.0038" ixy="0" ixz="0" iyy="0.0064" iyz="0" izz="0.0038"/></inertial>
@@ -44,5 +27,4 @@
   <xacro:macro name="SwerveWheelRight" params="position_name x_pos y_pos">
     <link name="${position_name}_steering_link">
-      <visual><origin/><geometry><mesh filename="package://antbot_description/meshes/steering_link_r.stl" scale="${steering_mesh_scale} ${steering_mesh_scale} ${steering_mesh_scale}"/></geometry><material name="metal_gray"/></visual>
       <collision><origin xyz="0 0.020 0.035"/><geometry><box size="0.050 0.075 0.110"/></geometry></collision>
       <inertial><mass value="1.0"/><origin xyz="0 0.020 0.035"/><inertia ixx="0.0017" ixy="0" ixz="0" iyy="0.0014" iyz="0" izz="0.0008"/></inertial>
@@ -54,6 +36,4 @@
     </joint>
     <link name="${position_name}_wheel_link">
-      <visual><origin/><geometry><mesh filename="package://antbot_description/meshes/wheel_link_r.stl" scale="${wheel_mesh_scale} ${wheel_mesh_scale} ${wheel_mesh_scale}"/></geometry><material name="tire_black"/></visual>
-      <xacro:WheelHub face_y="-0.035"/>
       <collision><origin rpy="${-pi/2} 0 0"/><geometry><cylinder radius="${wheel_radius}" length="${wheel_width}"/></geometry></collision>
       <inertial><mass value="2.0"/><inertia ixx="0.0038" ixy="0" ixz="0" iyy="0.0064" iyz="0" izz="0.0038"/></inertial>
@@ -64,8 +44,3 @@
     </joint>
   </xacro:macro>
-  <material name="tire_black"><color rgba="0.020 0.022 0.025 1.0"/></material>
-  <material name="metal_gray"><color rgba="0.42 0.44 0.47 1.0"/></material>
-  <material name="hub_silver"><color rgba="0.66 0.68 0.71 1.0"/></material>
-  <material name="hub_light"><color rgba="0.82 0.83 0.84 1.0"/></material>
-  <material name="hub_bolt_dark"><color rgba="0.25 0.27 0.29 1.0"/></material>
 </robot>
