Commit message: Update forearm vision diagnostics and robot workspace

File: dual_arm_ws/src/piper_h_description/urdf/piper_h_description.urdf (robot description, URDF)
Before this commit: robot piper_h_description, 7 links, 6 joints
Links:
- link Link1: mass 0.095130320813071 -> 0.71; geometry collision mesh filename=package://piper_h_description/meshes/Link1.STL; visual mesh filename=package://piper_h_description/meshes/dae/link1.dae
- link Link2: mass 0.297349969020434 -> 1.16; geometry collision mesh filename=package://piper_h_description/meshes/Link2.STL; visual mesh filename=package://piper_h_description/meshes/dae/link2.dae
- link Link3: mass 0.139005088174055 -> 0.5; geometry collision mesh filename=package://piper_h_description/meshes/Link3.STL; visual mesh filename=package://piper_h_description/meshes/dae/link3.dae
- link Link4: mass 0.0625155037542606 -> 0.38; geometry collision mesh filename=package://piper_h_description/meshes/Link4.STL; visual mesh filename=package://piper_h_description/meshes/dae/link4.dae
- link Link5: mass 0.0683301439531726 -> 0.39; geometry collision mesh filename=package://piper_h_description/meshes/Link5.STL; visual mesh filename=package://piper_h_description/meshes/dae/link5.dae
- link Link6: mass 0.851169543242842 -> 0.007; geometry collision mesh filename=package://piper_h_description/meshes/Link6.STL; visual mesh filename=package://piper_h_description/meshes/dae/link6.dae
- link base_link: mass 0.17076936349368 -> 1.02; geometry collision mesh filename=package://piper_h_description/meshes/base_link.STL; visual mesh filename=package://piper_h_description/meshes/dae/base_link.dae
Joints:
- joint joint1: limit lower=-2.618 upper=2.618 effort=100 velocity=3 -> lower=-2.6179938 upper=2.6179938 effort=100 velocity=5
- joint joint2: limit lower=0 upper=3.14 effort=100 velocity=3 -> lower=0 upper=3.1415926 effort=100 velocity=5; origin xyz=0 0 0 rpy=1.5708 -0.13674 3.1416 -> xyz=0 0 0 rpy=1.5707963 -0.1357866 -3.1415926
- joint joint3: limit lower=-2.96706 upper=0 effort=100 velocity=3 -> lower=-2.9670597 upper=0 effort=100 velocity=5; origin xyz=0.28508 0 0 rpy=0 0 -1.8796 -> xyz=0.28503 0 0 rpy=0 0 -1.7938494
- joint joint4: axis -0.087161 0 0.99619 -> 0 0 1; limit lower=-2.356195 upper=2.356195 effort=100 velocity=3 -> lower=-2.3561944 upper=2.3561944 effort=100 velocity=5; origin xyz=0 -0.25666 0 rpy=1.5708 0 0.17203 -> xyz=-0.02198 -0.25575 0 rpy=1.5707963 0 0
- joint joint5: limit lower=-1.56207 upper=1.56207 effort=100 velocity=3 -> lower=-1.5620696 upper=1.5620696 effort=100 velocity=5; origin xyz=0 0 0 rpy=-1.5708 -0.087272 0 -> xyz=0 0 0 rpy=-1.5707963 0 0
- joint joint6: axis -0.087161 0 0.99619 -> 0 0 1; limit lower=-3.14 upper=3.14 effort=100 velocity=3 -> lower=-2.0943951 upper=2.0943951 effort=100 velocity=5; origin xyz=0 -0.096 0 rpy=1.5708 0 0.087272 -> xyz=0 -0.0963 0 rpy=1.5707963 0 0
